File: pcb/left.kicad_sch (KiCad schematic)
At the start: 73 parts, among them J1 AudioJack3, SW1 TAB, SW10 D, SW11 F, SW12 G, SW13 CTRL, SW14 Z, SW15 X, SW16 C, SW17 V, SW18 B, SW19 META, SW2 Q, SW20 MOD, SW21 SPACE, SW3 W, SW4 E, SW43 Vertical Encoder, SW44 Horizontal Encoder, SW45 EX1, SW46 EX2, SW5 R, SW6 T, SW7 SHIFT, SW8 A, SW9 S

Commit message: Rework edgecuts and change to waveshare rp2040 zero
Parts:
- removed OL1: OLED, oled:SSD1306-0.91-OLED-4pin-128x32, symbol kbd:OLED
- removed SW43: Vertical Encoder, encoders:PEC12R-4220F-20024, symbol Device:RotaryEncoder_Switch
- removed SW44: Horizontal Encoder, encoders:PEC12R-2120F-S0012, symbol Device:RotaryEncoder_Switch
- added U1: RP2040-Zero, RP2040-Zero:RP2040-Zero, symbol RP2040-Zero:RP2040-Zero
- J1: footprint audio-jacks:PJ-399B-6A -> trs-jack:CUI_SJ-3501-SMT-TR; symbol Connector_Audio:AudioJack3 -> trsJack:SJ-3501-SMT-TR; MANUFACTURER (none) -> CUI Devices; MAXIMUM_PACKAGE_HEIGHT (none) -> 2.5mm; PARTREV (none) -> 1.05; STANDARD (none) -> Manufacturer Recommendations
Connections:
- net +5V: now also D43.1 (VDD), D46.1 (VDD), D47.1 (VDD), D48.1 (VDD), D49.1 (VDD), D50.1 (VDD), D51.1 (VDD), D52.1 (VDD), D53.1 (VDD), D54.1 (VDD), D55.1 (VDD), D56.1 (VDD), D57.1 (VDD), D58.1 (VDD), D59.1 (VDD), D60.1 (VDD), D61.1 (VDD), D62.1 (VDD), D63.1 (VDD), D64.1 (VDD), D65.1 (VDD), D66.1 (VDD), D67.1 (VDD), J1.3, U1.5v
- net COL_0: now also U1.15
- net COL_1: now also U1.26
- net COL_2: now also U1.27
- net COL_3: now also U1.28
- net COL_4: now also U1.14
- net COL_5: now also U1.13
- net COL_6: now also U1.29
- net GND: now also J1.1, J1.5, U1.GND; no longer J1.S
- net LED_GPIO: now also U1.8
- net ROW_0: now also U1.12
- net ROW_1: now also U1.11
- net ROW_2: now also U1.10
- net ROW_3: now also U1.9
- net TX: now also J1.2, J1.4, U1.0; no longer J1.R
- removed net 5v: D43.1 (VDD), D46.1 (VDD), D47.1 (VDD), D48.1 (VDD), D49.1 (VDD), D50.1 (VDD), D51.1 (VDD), D52.1 (VDD), D53.1 (VDD), D54.1 (VDD), D55.1 (VDD), D56.1 (VDD), D57.1 (VDD), D58.1 (VDD), D59.1 (VDD), D60.1 (VDD), D61.1 (VDD), D62.1 (VDD), D63.1 (VDD), D64.1 (VDD), D65.1 (VDD), D66.1 (VDD), D67.1 (VDD), J1.T
Other:
- removed sheet Left Pico

Commit message: Finalize pcb for printing
Connections:
- net COL_0: now also U1.13; no longer U1.15
- net COL_1: now also U1.14; no longer U1.26
- net COL_2: now also U1.15; no longer U1.27
- net COL_3: now also U1.26; no longer U1.28
- net COL_4: now also U1.27; no longer U1.14
- net COL_5: now also U1.12; no longer U1.13
- net ROW_0: now also U1.28; no longer U1.12
Changed lines of the file:
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@@
 	)
 	(label "COL_1"
-		(at 52.07 120.65 0)
-		(effects
-			(font
-				(size 1.27 1.27)
-			)
-			(justify left bottom)
-		)
-	)
-	(label "COL_5"
-		(at 52.07 113.03 0)
+		(at 52.07 115.57 0)
+		(effects
+			(font
+				(size 1.27 1.27)
+			)
+			(justify left bottom)
+		)
+	)
+	(label "COL_5"
+		(at 52.07 110.49 0)
 		(effects
 			(font
@@
 	)
 	(label "COL_4"
-		(at 52.07 115.57 0)
+		(at 52.07 123.19 0)
 		(effects
 			(font
@@
 	)
 	(label "ROW_0"
-		(at 52.07 110.49 0)
+		(at 52.07 125.73 0)
 		(effects
 			(font
@@
 	)
 	(label "COL_0"
-		(at 52.07 118.11 0)
+		(at 52.07 113.03 0)
 		(effects
 			(font
@@
 	)
 	(label "COL_2"
-		(at 52.07 123.19 0)
+		(at 52.07 118.11 0)
 		(effects
 			(font
@@
 	)
 	(label "COL_3"
-		(at 52.07 125.73 0)
-		(effects
-			(font
+		(at 52.07 120.65 0)
+		(effects
+			(font
