File: pcb/travyboard.kicad_pcb (KiCad board)
At the start: 2 copper layers, 360.2 x 95 mm, 210 parts, among them J1 AudioJack3, J2 AudioJack3, J3 USB_C_Receptacle_USB2.0_16P, J4 USB_C_Receptacle_USB2.0_16P, SW1 TAB, SW10 D, SW11 F, SW12 G, SW13 CTRL, SW14 Z, SW15 X, SW16 C, SW17 V, SW18 B, SW19 META, SW2 Q, SW20 MOD, SW21 SPACE, SW22 Y, SW23 U, SW24 I, SW25 O, SW26 P, SW27 BS, SW28 H, SW29 J, SW3 W, SW30 K, SW31 L, SW32 ;, SW33 ENTER, SW34 N, SW35 M, SW36 ,, SW37 ., SW38 /, SW39 SHIFT, SW4 E, SW40 META, SW41 MOD, SW42 SPACE, SW43 Vertical Encoder, SW44 Horizontal Encoder, SW45 EX1, SW46 EX2, SW47 Vertical Encoder, SW48 Horizontal Encoder, SW49 EX3, SW5 R, SW50 EX4, SW6 T, SW7 SHIFT, SW8 A, SW9 S, U2 W25Q128JVS, U3 RP2040, U4 NCP1117-1.5_SOT223, U5 TPD4E05U06DQA, U6 W25Q128JVS, U7 TPD4E05U06DQA, U8 NCP1117-1.5_SOT223, U9 RP2040, Y1 Crystal_GND24, Y2 Crystal_GND24

Commit message: Rework edgecuts and change to waveshare rp2040 zero
Parts:
- removed C1, C10, C11, C22, C23, C26, C27, C28, C29, C3, C30, C31, C32, C5, C6, C7, C8, C9: 100n, Capacitor_SMD:C_0402_1005Metric
- removed C12, C13, C18, C19: 10u, Capacitor_SMD:C_0402_1005Metric
- removed C14, C17, C2, C24, C25, C4: 1u, Capacitor_SMD:C_0402_1005Metric
- removed C15, C16, C20, C21: 27p, Capacitor_SMD:C_0402_1005Metric
- removed D93, D94: D, Diode_SMD:D_SOD-523
- removed J3, J4: USB_C_Receptacle_USB2.0_16P, usbc:TYPE-C-31-M-13C
- removed OL1, OL2: OLED, oled:SSD1306-0.91-OLED-4pin-128x32
- removed R1, R12, R13, R2: 5.1k, Resistor_SMD:R_0402_1005Metric
- removed R10, R16, R5, R9: 1k, Resistor_SMD:R_0402_1005Metric
- removed R11, R15, R4, R8: 10k, Resistor_SMD:R_0402_1005Metric
- removed R14, R3: 5.6k, Resistor_SMD:R_0402_1005Metric
- removed R17, R18, R6, R7: 27, Resistor_SMD:R_0402_1005Metric
- removed SW43, SW47: Vertical Encoder, encoders:PEC12R-4220F-20024
- removed SW44, SW48: Horizontal Encoder, encoders:PEC12R-2120F-S0012
- removed U3, U9: RP2040, Package_DFN_QFN:QFN-56-1EP_7x7mm_P0.4mm_EP3.2x3.2mm
- removed U4, U8: NCP1117-1.5_SOT223, Package_TO_SOT_SMD:SOT-223-3_TabPin2
- removed U5, U7: TPD4E05U06DQA, Package_SON:USON-10_2.5x1.0mm_P0.5mm
- removed U6: W25Q128JVS, Package_SO:SOIC-8_5.23x5.23mm_P1.27mm
- removed Y1, Y2: Crystal_GND24, Crystal:Crystal_SMD_3225-4Pin_3.2x2.5mm
- added U1: RP2040-Zero, RP2040-Zero:RP2040-Zero, F.Cu at (159.8, 71.9)
- J1, J2: footprint audio-jacks:PJ-399B-6A -> trs-jack:CUI_SJ-3501-SMT-TR; moved to B.Cu
- U2: value W25Q128JVS -> RP2040-Zero; footprint Package_SO:SOIC-8_5.23x5.23mm_P1.27mm -> RP2040-Zero:RP2040-Zero; moved to F.Cu
- moved U2 83.5 mm to (221.0, 72.0), turned to 0 degrees
- moved D20 28.3 mm to (254.7, 35.8)
- moved D21 28.3 mm to (273.7, 33.4)
- moved D22 28.3 mm to (292.8, 35.8)
- moved D23 28.3 mm to (311.8, 40.5)
- moved D24 28.3 mm to (330.9, 40.5)
- moved D26 28.3 mm to (254.7, 54.8)
- moved D27 28.3 mm to (273.7, 52.4)
- moved D28 28.3 mm to (292.8, 54.8)
- moved D29 28.3 mm to (311.8, 59.6)
- moved D30 28.3 mm to (330.9, 59.6)
- moved D32 28.3 mm to (254.7, 73.9)
- moved D33 28.3 mm to (273.7, 71.5)
- moved D34 28.3 mm to (292.8, 73.9)
- moved D35 28.3 mm to (311.8, 78.6)
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Connections:
- D43 pad 1: /Left Half/5v -> +5V
- D46 pad 1: /Left Half/5v -> +5V
- D47 pad 1: /Left Half/5v -> +5V
- D48 pad 1: /Left Half/5v -> +5V
- D49 pad 1: /Left Half/5v -> +5V
- D50 pad 1: /Left Half/5v -> +5V
- D51 pad 1: /Left Half/5v -> +5V
- D52 pad 1: /Left Half/5v -> +5V
- D53 pad 1: /Left Half/5v -> +5V
- D54 pad 1: /Left Half/5v -> +5V
- D55 pad 1: /Left Half/5v -> +5V
- D56 pad 1: /Left Half/5v -> +5V
- D57 pad 1: /Left Half/5v -> +5V
- D58 pad 1: /Left Half/5v -> +5V
- D59 pad 1: /Left Half/5v -> +5V
- D60 pad 1: /Left Half/5v -> +5V
- D61 pad 1: /Left Half/5v -> +5V
- D62 pad 1: /Left Half/5v -> +5V
- D63 pad 1: /Left Half/5v -> +5V
- D64 pad 1: /Left Half/5v -> +5V
- D65 pad 1: /Left Half/5v -> +5V
- D66 pad 1: /Left Half/5v -> +5V
- D67 pad 1: /Left Half/5v -> +5V
- D68 pad 1: /Right Half/5v -> +5V
- D68 pad 3: /Right Half/GND -> GND
- D69 pad 1: /Right Half/5v -> +5V
- D69 pad 3: /Right Half/GND -> GND
- D70 pad 1: /Right Half/5v -> +5V
- D70 pad 3: /Right Half/GND -> GND
- D71 pad 1: /Right Half/5v -> +5V
- D71 pad 3: /Right Half/GND -> GND
- D72 pad 1: /Right Half/5v -> +5V
- D72 pad 3: /Right Half/GND -> GND
- D73 pad 1: /Right Half/5v -> +5V
- D73 pad 3: /Right Half/GND -> GND
- D74 pad 1: /Right Half/5v -> +5V
- D74 pad 3: /Right Half/GND -> GND
- D75 pad 1: /Right Half/5v -> +5V
- D75 pad 3: /Right Half/GND -> GND
- D76 pad 1: /Right Half/5v -> +5V
- D76 pad 3: /Right Half/GND -> GND
- D77 pad 1: /Right Half/5v -> +5V
- D77 pad 3: /Right Half/GND -> GND
- D78 pad 1: /Right Half/5v -> +5V
- D78 pad 3: /Right Half/GND -> GND
- D79 pad 1: /Right Half/5v -> +5V
- D79 pad 3: /Right Half/GND -> GND
- D80 pad 1: /Right Half/5v -> +5V
- D80 pad 3: /Right Half/GND -> GND
- D81 pad 1: /Right Half/5v -> +5V
- D81 pad 3: /Right Half/GND -> GND
- D82 pad 1: /Right Half/5v -> +5V
- D82 pad 3: /Right Half/GND -> GND
- D83 pad 1: /Right Half/5v -> +5V
- D83 pad 3: /Right Half/GND -> GND
- D84 pad 1: /Right Half/5v -> +5V
- D84 pad 3: /Right Half/GND -> GND
- D85 pad 1: /Right Half/5v -> +5V
- D85 pad 3: /Right Half/GND -> GND
- D86 pad 1: /Right Half/5v -> +5V
- D86 pad 3: /Right Half/GND -> GND
- D87 pad 1: /Right Half/5v -> +5V
- D87 pad 3: /Right Half/GND -> GND
- D88 pad 1: /Right Half/5v -> +5V
- D88 pad 3: /Right Half/GND -> GND
- D89 pad 1: /Right Half/5v -> +5V
- D89 pad 3: /Right Half/GND -> GND
- D90 pad 1: /Right Half/5v -> +5V
- D90 pad 3: /Right Half/GND -> GND
- SW35 pad 2: unconnected-(SW35-Pad2) -> /Right Half/COL_2
- SW36 pad 2: unconnected-(SW36-Pad2) -> /Right Half/COL_3
- SW37 pad 2: unconnected-(SW37-Pad2) -> /Right Half/COL_4
- SW38 pad 2: unconnected-(SW38-Pad2) -> /Right Half/COL_5
- SW39 pad 2: unconnected-(SW39-Pad2) -> /Right Half/COL_6
- U2 pad 1: /Left Half/Left Pico/QSPI_SS -> /Right Half/RX
- U2 pad 2: /Left Half/Left Pico/QSPI_SD1 -> /Right Half/ROW_0
- U2 pad 3: /Left Half/Left Pico/QSPI_SD2 -> /Right Half/ROW_1
- U2 pad 4: GND -> /Right Half/COL_0
- U2 pad 5: /Left Half/Left Pico/QSPI_SD0 -> unconnected-(U2-Pad5)
- U2 pad 6: /Left Half/Left Pico/QSPI_SCLK -> unconnected-(U2-Pad6)
- U2 pad 7: /Left Half/Left Pico/QSPI_SD3 -> /Right Half/COL_1
- U2 pad 8: +3V3 -> /Right Half/COL_2
Routing:
- net /Right Half/COL_6: track 0.00 -> 166.2 mm, vias 0 -> 4
- net /Right Half/ROW_0: track 0.00 -> 157.3 mm, vias 0 -> 13
- net /Right Half/COL_5: track 0.00 -> 143.6 mm, vias 0 -> 4
- net /Right Half/ROW_1: track 0.00 -> 132.5 mm, vias 0 -> 11
- net /Right Half/COL_3: track 0.00 -> 128.3 mm, vias 0 -> 6
- net /Right Half/COL_4: track 0.00 -> 121.0 mm, vias 0 -> 4
- net /Right Half/ROW_2: track 0.00 -> 112.0 mm, vias 0 -> 8
- net /Right Half/COL_2: track 0.00 -> 110.3 mm, vias 0 -> 6
- net /Right Half/COL_1: track 0.00 -> 97.7 mm, vias 0 -> 6
- net /Right Half/ROW_3: track 0.00 -> 76.5 mm, vias 0 -> 3
- net +5V: track 0.00 -> 72.2 mm, vias 0 -> 37
- net Net-(D80-DOUT): track 0.00 -> 67.3 mm, vias 0 -> 2
- net /Right Half/COL_0: track 0.00 -> 44.2 mm, vias 0 -> 3
- net Net-(D70-DOUT): track 0.00 -> 40.3 mm
- net Net-(D72-DIN): track 0.00 -> 33.8 mm, vias 0 -> 2
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- added copper zone on F.Cu, net +5V
- added copper zone on B.Cu, net GND
Other:
- board size 360.2 x 95 mm -> 314.3 x 92.6 mm

Commit message: Finalize pcb for printing
Parts:
- added mouse-bite-5mm-10mm: VAL**, mouseBites:mouse-bite-5mm-10mm, F.Cu at (191.9, 21.3)
- added mouse-bite-5mm-10mm: VAL**, mouseBites:mouse-bite-5mm-10mm, F.Cu at (53.1, 85.8)
- added mouse-bite-5mm-10mm: VAL**, mouseBites:mouse-bite-5mm-10mm, F.Cu at (80.9, 18.9)
- added mouse-bite-5mm-10mm: VAL**, mouseBites:mouse-bite-5mm-10mm, F.Cu at (298.7, 85.8)
- added mouse-bite-5mm-10mm: VAL**, mouseBites:mouse-bite-5mm-10mm, F.Cu at (160.0, 21.3)
- added mouse-bite-5mm-10mm: VAL**, mouseBites:mouse-bite-5mm-10mm, F.Cu at (271.1, 18.9)
- moved D19 28.8 mm to (206.8, 38.1)
- moved D20 28.8 mm to (225.9, 35.8)
- moved D22 28.8 mm to (264.0, 35.8)
- moved D24 28.8 mm to (302.1, 40.5)
- moved D25 28.8 mm to (206.8, 57.2)
- moved D26 28.8 mm to (225.9, 54.8)
- moved D28 28.8 mm to (264.0, 54.8)
- moved D30 28.8 mm to (302.1, 59.6)
- moved D31 28.8 mm to (206.8, 76.2)
- moved D32 28.8 mm to (225.9, 73.9)
- moved D34 28.8 mm to (264.0, 73.9)
- moved D36 28.8 mm to (302.1, 78.6)
- moved D40 28.8 mm to (197.2, 106.4)
- moved D41 28.8 mm to (215.7, 98.9)
- moved D42 28.8 mm to (235.4, 95.3)
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Connections:
- U1 pad 12: /Left Half/ROW_0 -> /Left Half/COL_5
- U1 pad 13: /Left Half/COL_5 -> /Left Half/COL_0
- U1 pad 14: /Left Half/COL_4 -> /Left Half/COL_1
- U1 pad 15: /Left Half/COL_0 -> /Left Half/COL_2
- U1 pad 26: /Left Half/COL_1 -> /Left Half/COL_3
- U1 pad 27: /Left Half/COL_2 -> /Left Half/COL_4
- U1 pad 28: /Left Half/COL_3 -> /Left Half/ROW_0
Routing:
- net /Left Half/ROW_0: track 0.00 -> 154.5 mm, vias 0 -> 10
- net /Left Half/ROW_1: track 0.10 -> 150.3 mm, vias 0 -> 12
- net /Left Half/COL_0: track 3.06 -> 146.3 mm, vias 0 -> 4
- net /Left Half/ROW_2: track 0.09 -> 136.0 mm, vias 0 -> 6
- net /Left Half/COL_1: track 3.05 -> 126.2 mm, vias 0 -> 4
- net /Left Half/COL_3: track 3.05 -> 119.1 mm, vias 0 -> 6
- net /Left Half/COL_2: track 3.52 -> 107.8 mm, vias 0 -> 4
- net /Left Half/COL_4: track 3.90 -> 103.6 mm, vias 0 -> 6
- net /Left Half/COL_5: track 5.15 -> 83.3 mm, vias 0 -> 6
- net /Left Half/ROW_3: track 0.00 -> 75.9 mm, vias 0 -> 3
- net Net-(D47-DOUT): track 0.00 -> 38.9 mm, vias 0 -> 2
- net /Left Half/COL_6: track 2.29 -> 39.4 mm
- net Net-(D60-DOUT): track 0.00 -> 28.8 mm, vias 0 -> 2
- net Net-(D49-DOUT): track 0.00 -> 28.0 mm
- net Net-(D63-DOUT): track 0.00 -> 28.0 mm
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Other:
- board size 314.3 x 92.6 mm -> 285.5 x 106.3 mm
- board text added: "JLCJLCJLCJLC"
- board text added: "travyboard v1"

Commit message: Remove kicad backups from git
Parts:
- moved D29 15.1 mm to (280.6, 74.5)
- moved D35 15.1 mm to (280.6, 93.5)
- moved D42 15.1 mm to (233.0, 110.2)
- moved D76 15.1 mm to (306.8, 76.2)
- moved D82 15.1 mm to (287.8, 76.2)
- moved D87 15.1 mm to (287.8, 95.3)
- moved SW25 15.1 mm to (268.7, 45.8)
- moved SW27 15.1 mm to (306.8, 50.6)
- moved SW31 15.1 mm to (268.7, 64.9)
- moved SW37 15.1 mm to (268.7, 83.9)
- moved mouse-bite-5mm-10mm 15.1 mm to (268.7, 33.8)
- moved D12 15.1 mm to (128.4, 72.1)
- moved D13 15.1 mm to (33.2, 93.5)
- moved D14 15.1 mm to (52.2, 93.5)
- moved D15 15.1 mm to (71.3, 88.7)
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